File: hifi-cab.kicad_pcb (KiCad board)
At the start: 2 copper layers, 28 parts, among them J10 BUTTON, J11 RS-232, J13 PWR IN, J3 FAN 1, J6 FAN 2, J7 IR REMOTE, J8 DS18B20, J9 DS18B20, Q1 AO3400A, Q2 AO3400A, Q3 AO3400A, U1 esp32-wemos-d1-mini, U2 TSR0.5-2433

Commit message: Default to old habits.
Parts:
- removed ?: , 
- moved C1 54.4 mm to (112.5, 94.4)
- moved J8 40.8 mm to (98.8, 166.7)
- moved J9 40.8 mm to (98.8, 174.0)
- moved R10 40.8 mm to (97.7, 160.7)
- moved J3 31.4 mm to (136.0, 97.3), turned to -90 degrees
- moved D2 23.9 mm to (128.0, 97.3), turned to 180 degrees
- moved J6 21.0 mm to (136.0, 111.3), turned to -90 degrees
- moved R3 17.6 mm to (128.4, 103.4), turned to -90 degrees
- moved R6 15.1 mm to (128.4, 117.4), turned to -90 degrees
- moved J10 14.7 mm to (95.0, 138.8)
- moved R11 14.7 mm to (98.5, 132.8)
- moved J13 14.6 mm to (85.7, 138.8)
- moved R5 13.8 mm to (115.7, 117.4), turned to 90 degrees
- moved Q1 13.3 mm to (123.2, 103.2), turned to 0 degrees
- moved R2 12.7 mm to (115.7, 103.3), turned to 90 degrees
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Routing:
- net VCC: track 124.0 -> 64.0 mm
- net +3.3V: track 21.6 -> 34.7 mm

Commit message: Enough for tonight.
Parts:
- moved J9 35.6 mm to (104.2, 138.8)
- moved J8 32.5 mm to (115.5, 138.8)
- moved R10 28.7 mm to (104.2, 132.8)
- moved Q2 13.3 mm to (120.1, 126.6), turned to 90 degrees
- moved R9 10.7 mm to (129.2, 125.4), turned to 180 degrees
- moved R7 10.6 mm to (117.8, 131.4), turned to 90 degrees
- moved J7 8.36 mm to (135.1, 132.9), turned to 90 degrees
- moved R8 6.27 mm to (121.8, 131.4), turned to 90 degrees
Routing:
- net +3.3V: track 34.7 -> 27.4 mm
- net DS18B20: track 7.32 -> 0.00 mm
- net IR_1: track 3.44 -> 0.00 mm
