File: hifi-cab.kicad_pcb (KiCad board)
At the start: 2 copper layers, 102 x 58 mm, 29 parts, among them J1 FAN 1, J2 FAN 2, J3 FAN 3, J4 IR LED, J5 DS18B20, J6 PWR IN, J7 IR LED, K1 FAN RELAY, K2 FAN RELAY, K3 FAN RELAY, Q1 2N3904, Q2 2N3904, Q3 2N3904, Q4 2N3904, U1 ESP32 D1 MINI, U3 TSR0.5-2433

Commit message: Update hifi-cab.kicad_pcb
Routing:
- net IR: track 7.05 -> 35.2 mm
- net TACH3: track 18.8 -> 30.8 mm
- net RPM3: track 17.1 -> 29.1 mm
- net TACH2: track 18.8 -> 30.7 mm
- net TACH1: track 18.8 -> 30.6 mm
- net RPM2: track 17.1 -> 28.9 mm
- net RPM1: track 17.1 -> 28.9 mm
- net VCC: track 162.9 -> 174.4 mm
- net RELAY3: track 20.2 -> 9.10 mm
- net +3.3V: track 141.8 -> 146.8 mm, vias 0 -> 1
Changed lines of the file:
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@@
+	)
+	(segment
+		(start 119.48 52.03)
+		(end 122.9 55.45)
+		(width 0.5)
+		(layer "F.Cu")
+		(net "+3.3V")
+	)
+	(segment
+		(start 119.48 49.32)
+		(end 119.48 52.03)
+		(width 0.5)
+		(layer "F.Cu")
+		(net "+3.3V")
+	)
+	(via
+		(at 122.9 55.45)
+		(size 0.6)
+		(drill 0.3)
+		(layers "F.Cu" "B.Cu")
+		(net "+3.3V")
 	)
 	(segment
@@
 	)
 	(segment
-		(start 132.7 49.4)
-		(end 89.36 49.4)
-		(width 0.5)
-		(layer "B.Cu")
-		(net "+3.3V")
-	)
-	(segment
 		(start 139.4 70.1)
 		(end 132.68 63.38)
@@
 	)
 	(segment
+		(start 122.9 55.45)
+		(end 130.78 55.45)
+		(width 0.5)
+		(layer "B.Cu")
+		(net "+3.3V")
+	)
+	(segment
 		(start 159.1 80.85)
 		(end 159.1 74.7)
@@
 	)
 	(segment
+		(start 119.48 49.32)
+		(end 89.28 49.32)
+		(width 0.5)
+		(layer "B.Cu")
+		(net "+3.3V")
+	)
+	(segment
 		(start 159.1 62.65)
 		(end 153.560056 57.110056)
@@
 	)
 	(segment
+		(start 130.78 55.45)
+		(end 132.68 57.35)
+		(width 0.5)
+		(layer "B.Cu")
+		(net "+3.3V")
+	)
+	(segment
 		(start 159.1 74.7)
 		(end 154.5 70.1)
@@
 	)
 	(segment
+		(start 132.68 57.35)
+		(end 132.68 63.38)
+		(width 1)
+		(layer "B.Cu")
+		(net "+3.3V")
+	)
+	(segment
 		(start 132.68 50.08)
-		(end 132.68 63.38)
+		(end 132.68 57.35)
 		(width 1)
 		(layer "B.Cu")
@@
 	)
 	(segment
+		(start 132.7 44.32)
+		(end 132.56 44.32)
+		(width 1)
+		(layer "B.Cu")
+		(net "VCC")
+	)
+	(segment
 		(start 83.182379 52.3)
 		(end 82.882379 52)
@@
 	)
 	(segment
+		(start 132.56 44.32)
+		(end 124.58 52.3)
+		(width 1)
+		(layer "B.Cu")
+		(net "VCC")
+	)
+	(segment
 		(start 132.68 35.87)
 		(end 132.75 35.8)
@@
 	)
 	(segment
+		(start 122.4 58.2)
+		(end 122.4 62)
+		(width 0.5)
+		(layer "F.Cu")
+		(net "TACH3")
+	)
+	(segment
 		(start 116.585 44.615)
 		(end 116.585 52.385)
@@
 	)
 	(segment
+		(start 116.585 52.385)
+		(end 122.4 58.2)
+		(width 0.5)
+		(layer "F.Cu")
+		(net "TACH3")
+	)
+	(segment
 		(start 118.446 40.666)
 		(end 119.48 41.7)
@@
 	)
 	(segment
+		(start 161.3 71.6)
+		(end 167.2 65.7)
+		(width 0.5)
+		(layer "F.Cu")
+		(net "IR")
+	)
+	(segment
 		(start 140.41 78.94)
-		(end 143.3 76.05)
+		(end 147.75 71.6)
 		(width 0.5)
 		(layer "F.Cu")
@@
 	)
 	(segment
-		(start 127.4 79.81)
-		(end 127.4 62.6)
-		(width 0.5)
-		(layer "F.Cu")
-		(net "RELAY3")
-	)
-	(segment
-		(start 125.31 81.9)
-		(end 127.4 79.81)
+		(start 147.75 71.6)
+		(end 161.3 71.6)
+		(width 0.5)
+		(layer "F.Cu")
+		(net "IR")
+	)
+	(segment
+		(start 127.473 79.737)
+		(end 127.473 73.7)
 		(width 0.5)
 		(layer "F.Cu")
@@
 	)
 	(segment
+		(start 125.31 81.9)
+		(end 127.473 79.737)
+		(width 0.5)
+		(layer "F.Cu")
+		(net "RELAY3")
+	)
+	(segment
+		(start 86.32 52.193)
+		(end 92.135 58.008)
+		(width 0.5)
+		(layer "F.Cu")
+		(net "TACH1")
+	)
+	(segment
 		(start 86.35 44.63)
-		(end 86.35 52.4)
+		(end 86.35 52.163)
 		(width 0.5)
 		(layer "F.Cu")
@@
 	)
 	(segment
+		(start 92.135 58.008)
+		(end 92.135 61.808)
+		(width 0.5)
+		(layer "F.Cu")
+		(net "TACH1")
+	)
+	(segment
+		(start 86.35 52.163)
+		(end 86.32 52.193)
+		(width 0.5)
+		(layer "F.Cu")
+		(net "TACH1")
+	)
+	(segment
 		(start 89.32 35.7)
 		(end 88.266 36.754)
@@
 	)
 	(segment
+		(start 121.773 58.55)
+		(end 121.773 61.85)
+		(width 0.5)
+		(layer "F.Cu")
+		(net "RPM3")
+	)
+	(segment
+		(start 115.815 52.592)
+		(end 121.773 58.55)
+		(width 0.5)
+		(layer "F.Cu")
+		(net "RPM3")
+	)
+	(segment
+		(start 117.015 35.685)
+		(end 117.015 43.055)
+		(width 0.5)
+		(layer "F.Cu")
+		(net "RPM3")
+	)
+	(segment
 		(start 117.015 43.055)
 		(end 115.815 44.255)
@@
 	)
 	(segment
-		(start 117.015 35.685)
-		(end 117.015 43.055)
-		(width 0.5)
-		(layer "F.Cu")
-		(net "RPM3")
-	)
-	(segment
 		(start 115.815 44.255)
-		(end 115.815 52.315)
+		(end 115.815 52.592)
 		(width 0.5)
 		(layer "F.Cu")
@@
 	)
 	(segment
+		(start 100.75 52.5)
+		(end 106.708 58.458)
+		(width 0.5)
+		(layer "F.Cu")
+		(net "RPM2")
+	)
+	(segment
 		(start 101.965 43.105)
 		(end 100.765 44.305)
@@
 	)
 	(segment
+		(start 106.708 58.458)
+		(end 106.708 61.758)
+		(width 0.5)
+		(layer "F.Cu")
+		(net "RPM2")
+	)
+	(segment
 		(start 100.765 44.305)
 		(end 100.765 52.365)
@@
 	)
 	(segment
+		(start 91.508 58.358)
+		(end 91.508 61.658)
+		(width 0.5)
+		(layer "F.Cu")
+		(net "RPM1")
+	)
+	(segment
 		(start 85.58 44.27)
 		(end 85.58 52.33)
@@
 	)
 	(segment
+		(start 85.55 52.4)
+		(end 91.508 58.358)
+		(width 0.5)
+		(layer "F.Cu")
+		(net "RPM1")
+	)
+	(segment
 		(start 94.55 58.54)
 		(end 97.95 55.14)
@@
 	)
 	(segment
-		(start 101.535 44.665)
-		(end 101.535 52.435)
+		(start 101.535 52.278)
+		(end 101.52 52.293)
+		(width 0.5)
+		(layer "F.Cu")
+		(net "TACH2")
+	)
+	(segment
+		(start 101.52 52.293)
+		(end 107.335 58.108)
 		(width 0.5)
 		(layer "F.Cu")
@@
 		(width 0.5)
 		(layer "F.Cu")
+		(net "TACH2")
+	)
+	(segment
+		(start 101.535 44.665)
+		(end 101.535 52.278)
+		(width 0.5)
+		(layer "F.Cu")
+		(net "TACH2")
+	)
+	(segment
+		(start 107.335 58.108)
+		(end 107.335 61.908)
+		(width 0.5)
+		(layer "F.Cu")
