File: hifi-cab.kicad_sch (KiCad schematic)
At the start: 31 parts, among them J1 IR, J2 FAN 1, J3 FAN 2, J4 FAN 3, J5 DS18B20, J6 PWR IN, J7 RS-232, Q1 AO3400A, Q2 AO3400A, Q3 AO3400A, Q4 AO3400A, U1 TSR0.5-2433, U2 esp32-wemos-d1-mini

Commit message: Start fix for manufacturing defects
Parts:
- removed C2: 100nF, Capacitor_SMD:C_0805_2012Metric_Pad1.18x1.45mm_HandSolder, symbol Device:C
- removed J1: IR, Connector_JST:JST_XH_B2B-XH-A_1x02_P2.50mm_Vertical, symbol Connector:Conn_01x02_Pin
- removed J7: RS-232, Connector_JST:JST_XH_B4B-XH-A_1x04_P2.50mm_Vertical, symbol Connector:Conn_01x04_Pin
- removed Q1, Q2, Q3, Q4: AO3400A, Package_TO_SOT_SMD:SOT-23, symbol Transistor_FET:AO3400A
- removed R1: 10K, Resistor_SMD:R_0805_2012Metric_Pad1.20x1.40mm_HandSolder, symbol Device:R
- removed R10, R11: 680R, Resistor_SMD:R_0805_2012Metric_Pad1.20x1.40mm_HandSolder, symbol Device:R
- removed R6, R7, R8: 100R, Resistor_SMD:R_0805_2012Metric_Pad1.20x1.40mm_HandSolder, symbol Device:R
- removed R9: 68R, Resistor_THT:R_Axial_DIN0204_L3.6mm_D1.6mm_P5.08mm_Horizontal, symbol Device:R
- added D4: 1N4004, Diode_THT:D_DO-41_SOD81_P10.16mm_Horizontal, symbol Diode:1N4004
- added J7: FAN 3, Connector:FanPinHeader_1x04_P2.54mm_Vertical, symbol Connector:Screw_Terminal_01x04
- added K3, K4, K5: FAN RELAY, symbol Relay:Relay_SPDT
- added Q1, Q2, Q3: 2N3904, Package_TO_SOT_THT:TO-92_Inline, symbol Transistor_BJT:2N3904
- added R1: 1K6, Resistor_THT:R_Axial_DIN0204_L3.6mm_D1.6mm_P7.62mm_Horizontal, symbol Device:R
- added R1: 680R, Resistor_SMD:R_0805_2012Metric_Pad1.20x1.40mm_HandSolder, symbol Device:R
- R2, R4: value 10K -> 680R
- R3: value 10K -> 1K6; footprint Resistor_SMD:R_0805_2012Metric_Pad1.20x1.40mm_HandSolder -> Resistor_THT:R_Axial_DIN0204_L3.6mm_D1.6mm_P7.62mm_Horizontal
- R5: value 100R -> 1K6; footprint Resistor_SMD:R_0805_2012Metric_Pad1.20x1.40mm_HandSolder -> Resistor_THT:R_Axial_DIN0204_L3.6mm_D1.6mm_P7.62mm_Horizontal
Connections:
- net +3.3V: now also R2.2, R4.2, R1.2
- net FAN1_C: no longer R2.1
- net FAN2_C: no longer R3.1
- net FAN3_C: no longer R4.1
- net GND: now also K3.14, K4.14, K5.14, Q1.1 (E), Q2.1 (E), Q3.1 (E); no longer R2.2, R3.2, R4.2
- net IR_C: no longer R5.1
- net RPM3: now also J7.4 (Pin_4)
- net TACH1: now also R1.1
- net TACH2: now also R2.1
- net TACH3: now also R4.1, J7.3 (Pin_3)
- net VCC: now also K3.A2, K4.A2, K5.A2
- net RELAY3: now reaches R5.2
- net FAN1: no longer names the net of D1.1 (K), J2.1 (Pin_1)
- net FAN1: now also K3.11
- net FAN2: no longer names the net of D2.1 (K), J3.1 (Pin_1)
- net FAN2: now also K4.11
- net RX: no longer names the net of U2.23 (RXD)
- net TX: no longer names the net of U2.21 (TXD)
- new net: D4.1 (K), J7.1 (Pin_1), K5.11
- new net: K5.A1, Q3.3 (C)
- new net: D4.2 (A), J7.2 (Pin_2)
- new net: Q1.2 (B), R1.1
- new net: Q2.2 (B), R3.1
- new net: K4.A1, Q2.3 (C)
- new net: K3.A1, Q1.3 (C)
- new net: Q3.2 (B), R5.1
- new net RELAY1: R1.2
- new net RELAY2: R3.2
- no-connect marks 21 -> 26
Other:
- moved on the sheet: D3, J4, J5, R12, R13, U2

Commit message: Housekeeping
Parts:
- removed D3: 1N4004, Diode_THT:D_DO-41_SOD81_P10.16mm_Horizontal, symbol Diode:1N4004
- removed J4: FAN 3, Connector:FanPinHeader_1x04_P2.54mm_Vertical, symbol Connector:Screw_Terminal_01x04
- removed R12: 680R, Resistor_SMD:R_0805_2012Metric_Pad1.20x1.40mm_HandSolder, symbol Device:R
- U2: value esp32-wemos-d1-mini -> ESP32 D1 MINI
Connections:
- net DS18B20: no longer U2.6 (IO_26/D0)
- net RPM1: no longer U2.17 (IO_09/SD2)
- net RPM2: no longer U2.13 (IO_14/TMS)
- net RPM3: no longer U2.9 (IO_33)
- net TACH1: no longer U2.18 (IO_13/TCK)
- net TACH2: no longer U2.11 (IO_34)
- net TACH3: no longer U2.5 (IO_39/SVN)
- net VCC: now also D4.2 (A), J7.2 (Pin_2)
- net FAN1_C: no longer names the net of U2.8 (IO_18/D5)
- net FAN2_C: no longer names the net of U2.10 (IO_19/D6)
- net FAN3_C: no longer names the net of U2.12 (IO_23/D7)
- net IR_C: no longer names the net of U2.14 (IO_05/D8)
- no-connect marks 26 -> 3
Other:
- note added: "POWER RAILS"
- moved on the sheet: U2

Commit message: Layout v4
Parts:
- added J4: IR LED, Connector_JST:JST_XH_B2B-XH-A_1x02_P2.50mm_Vertical, symbol Connector:Conn_01x02_Pin
- added Q4: 2N3904, Package_TO_SOT_THT:TO-92_Inline, symbol Transistor_BJT:2N3904
- added R5: --, Resistor_THT:R_Axial_DIN0204_L3.6mm_D1.6mm_P7.62mm_Horizontal, symbol Device:R
- added R7: 1K6, Resistor_THT:R_Axial_DIN0204_L3.6mm_D1.6mm_P7.62mm_Horizontal, symbol Device:R
- added U2: CC1101, CC1101:CC1101, symbol custom:C1101
- K1: renamed from K3; footprint (none) -> SR5-12V-200-1C:RELAY_SR5-12V-200-1C
- K2: renamed from K4; footprint (none) -> SR5-12V-200-1C:RELAY_SR5-12V-200-1C
- K3: renamed from K5; footprint (none) -> SR5-12V-200-1C:RELAY_SR5-12V-200-1C
- R1: footprint Resistor_SMD:R_0805_2012Metric_Pad1.20x1.40mm_HandSolder -> Resistor_THT:R_Axial_DIN0204_L3.6mm_D1.6mm_P7.62mm_Horizontal
- R3: renamed from R2; footprint Resistor_SMD:R_0805_2012Metric_Pad1.20x1.40mm_HandSolder -> Resistor_THT:R_Axial_DIN0204_L3.6mm_D1.6mm_P7.62mm_Horizontal
- R6: renamed from R4; footprint Resistor_SMD:R_0805_2012Metric_Pad1.20x1.40mm_HandSolder -> Resistor_THT:R_Axial_DIN0204_L3.6mm_D1.6mm_P7.62mm_Horizontal
- R9: renamed from R13; footprint Resistor_SMD:R_0805_2012Metric_Pad1.20x1.40mm_HandSolder -> Resistor_THT:R_Axial_DIN0204_L3.6mm_D1.6mm_P7.62mm_Horizontal
- renumbered D4 to D3, J2 to J1, J3 to J2, J7 to J3, R1 to R2, R3 to R4, R5 to R8, U2 to U1, U1 to U3
Connections:
- net +3.3V: now also J4.1 (Pin_1), U2.2 (VCC)
- net GND: now also Q4.1 (E), U2.1 (GND)
- net MISO: now reaches U1.10 (IO_19/D6)
- net MISO: now also U2.7 (MISO)
- net MOSI: now reaches U1.12 (IO_23/D7)
- net MOSI: now also U2.6 (MOSI)
- net CSN: now reaches U1.14 (IO_05/D8)
- net CSN: now also U2.4 (CSN)
- net SCLK: now reaches U1.8 (IO_18/D5)
- net SCLK: now also U2.5 (SCLK)
- new net: Q4.2 (B), R7.1
- new net: Q4.3 (C), R5.2
- new net: J4.2 (Pin_2), R5.1
- new net IR: R7.2
- no-connect marks 3 -> 6
Other:
- note added: "DS18B20 TEMP SENSORS"
- note added: "IR BLASTER"
- note added: "POWER"
- note removed: "POWER RAILS"
- moved on the sheet: J5, R9

Commit message: Start routing power (it never ends)
Parts:
- R5: value -- -> 68R
Changed lines of the file:
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@@
 			)
 		)
-		(property "Value" "--"
+		(property "Value" "68R"
 			(at 199.39 130.81 90)
 			(show_name no)
